File: i2c_stepper_driver_breakout.sch (KiCad schematic (older format))
At the start: 13 parts, among them J1 Conn_01x10, J2 Conn_01x10, J3 S4B-PH-SM4-TB, U1 PCA9629A, U2 A3909

Commit message: Continued layout
Parts:
- added U3: MAX17291, Locator_Footprints:MAX17291ATA+T, symbol Locator_Library:MAX17291
- J3: value S4B-PH-SM4-TB -> B4B-PH-K-S; footprint Connector_JST:JST_PH_B4B-PH-K_1x04_P2.00mm_Vertical -> Locator_Footprints:JST_PH_S4B-PH-SM4-TB_1x04-1MP_P2.00mm_Horizontal
- R1, R2: value 10K -> DNP
- U2: footprint Package_SO:MSOP-10-1EP_3x3mm_P0.5mm_EP1.73x1.98mm_ThermalVias -> Locator_Footprints:A3909
Connections:
- net GND: now also J1.1 (Pin_1), J1.10 (Pin_10), J2.1 (Pin_1), J2.10 (Pin_10), U2.11 (PAD)
Other:
- note added: "5.5V Boost for logic and motor"
- note added: "JST Connector (Motor)"
- note removed: "JST Motor Connector"
- moved on the sheet: J1, J2
Changed lines of the file:
@@
 F 0 "U2" H 4225 2165 50  0000 C CNN
 F 1 "A3909" H 4225 2074 50  0000 C CNN
-F 2 "Package_SO:MSOP-10-1EP_3x3mm_P0.5mm_EP1.73x1.98mm_ThermalVias" H 4000 2050 50  0001 C CNN
+F 2 "Locator_Footprints:A3909" H 4000 2050 50  0001 C CNN
 F 3 "" H 4000 2050 50  0001 C CNN
 	1    3950 2000
@@
 I2C address: 40h
 $Comp
-L Connector_Generic:Conn_01x10 J1
-U 1 1 5FDC0F46
-P 7950 1950
-F 0 "J1" H 7900 2550 50  0000 C CNN
-F 1 "Conn_01x10" H 7900 2450 50  0000 C CNN
-F 2 "Connector_PinHeader_2.54mm:PinHeader_1x10_P2.54mm_Vertical" H 7950 1950 50  0001 C CNN
-F 3 "~" H 7950 1950 50  0001 C CNN
-	1    7950 1950
-	1    0    0    -1
-$EndComp
-$Comp
 L Connector_Generic:Conn_01x10 J2
 U 1 1 5FDC3C47
-P 8350 2050
-F 0 "J2" H 8350 1350 50  0000 C CNN
-F 1 "Conn_01x10" H 8300 1450 50  0000 C CNN
-F 2 "Connector_PinHeader_2.54mm:PinHeader_1x10_P2.54mm_Vertical" H 8350 2050 50  0001 C CNN
-F 3 "~" H 8350 2050 50  0001 C CNN
-	1    8350 2050
+P 8400 2050
+F 0 "J2" H 8400 1350 50  0000 C CNN
+F 1 "Conn_01x10" H 8350 1450 50  0000 C CNN
+F 2 "Connector_PinHeader_2.54mm:PinHeader_1x10_P2.54mm_Vertical" H 8400 2050 50  0001 C CNN
+F 3 "~" H 8400 2050 50  0001 C CNN
+	1    8400 2050
 	-1   0    0    1
 $EndComp
@@
 	9400 3300 9400 600
 Text Notes 9600 800  0    79   ~ 0
-JST Motor Connector
+JST Connector (Motor)
 $Comp
 L Device:R R2
@@
 P 1400 1250
 F 0 "R2" H 1470 1296 50  0000 L CNN
-F 1 "10K" H 1470 1205 50  0000 L CNN
+F 1 "DNP" H 1470 1205 50  0000 L CNN
 F 2 "Resistor_SMD:R_0402_1005Metric" V 1330 1250 50  0001 C CNN
 F 3 "~" H 1400 1250 50  0001 C CNN
@@
 P 1100 1250
 F 0 "R1" H 1170 1296 50  0000 L CNN
-F 1 "10K" H 1170 1205 50  0000 L CNN
+F 1 "DNP" H 1170 1205 50  0000 L CNN
 F 2 "Resistor_SMD:R_0402_1005Metric" V 1030 1250 50  0001 C CNN
 F 3 "~" H 1100 1250 50  0001 C CNN
@@
 Text Label 9800 1800 0    50   ~ 0
 OUT3
+Text Label 9800 2100 0    50   ~ 0
+OUT2
+Text Label 9800 2000 0    50   ~ 0
+OUT4
+$Comp
+L Connector_Generic:Conn_01x10 J1
+U 1 1 5FDC0F46
+P 8000 1950
+F 0 "J1" H 7950 2550 50  0000 C CNN
+F 1 "Conn_01x10" H 7950 2450 50  0000 C CNN
+F 2 "Connector_PinHeader_2.54mm:PinHeader_1x10_P2.54mm_Vertical" H 8000 1950 50  0001 C CNN
+F 3 "~" H 8000 1950 50  0001 C CNN
+	1    8000 1950
+	1    0    0    -1
+$EndComp
+Wire Wire Line
+	7800 1550 7350 1550
+Wire Wire Line
+	9050 1550 8600 1550
+$Comp
+L power:GND #PWR0106
+U 1 1 5FE434C6
+P 7350 1550
+F 0 "#PWR0106" H 7350 1300 50  0001 C CNN
+F 1 "GND" H 7355 1377 50  0000 C CNN
+F 2 "" H 7350 1550 50  0001 C CNN
+F 3 "" H 7350 1550 50  0001 C CNN
+	1    7350 1550
+	1    0    0    -1
+$EndComp
+$Comp
+L power:GND #PWR0107
+U 1 1 5FE43CDC
+P 9050 1550
+F 0 "#PWR0107" H 9050 1300 50  0001 C CNN
+F 1 "GND" H 9055 1377 50  0000 C CNN
+F 2 "" H 9050 1550 50  0001 C CNN
+F 3 "" H 9050 1550 50  0001 C CNN
+	1    9050 1550
+	1    0    0    -1
+$EndComp
+Wire Wire Line
+	9050 2450 8600 2450
+$Comp
+L power:GND #PWR0108
+U 1 1 5FE445F7
+P 9050 2450
+F 0 "#PWR0108" H 9050 2200 50  0001 C CNN
+F 1 "GND" H 9055 2277 50  0000 C CNN
+F 2 "" H 9050 2450 50  0001 C CNN
+F 3 "" H 9050 2450 50  0001 C CNN
+	1    9050 2450
+	1    0    0    -1
+$EndComp
+Wire Wire Line
+	7800 2450 7350 2450
+$Comp
+L power:GND #PWR0109
+U 1 1 5FE45CE7
+P 7350 2450
+F 0 "#PWR0109" H 7350 2200 50  0001 C CNN
+F 1 "GND" H 7355 2277 50  0000 C CNN
+F 2 "" H 7350 2450 50  0001 C CNN
+F 3 "" H 7350 2450 50  0001 C CNN
+	1    7350 2450
+	1    0    0    -1
+$EndComp
+$Comp
+L Locator_Library:MAX17291 U3
+U 1 1 5FE52B80
+P 2550 4500
+F 0 "U3" H 2950 4781 50  0000 C CNN
+F 1 "MAX17291" H 2950 4690 50  0000 C CNN
+F 2 "Locator_Footprints:MAX17291ATA+T" H 2600 4550 50  0001 C CNN
+F 3 "" H 2600 4550 50  0001 C CNN
+	1    2550 4500
+	1    0    0    -1
+$EndComp
 $Comp
 L Connector_Generic:Conn_01x04 J3
@@
 P 10250 1900
 F 0 "J3" H 10330 1892 50  0000 L CNN
-F 1 "S4B-PH-SM4-TB" H 10330 1801 50  0000 L CNN
-F 2 "Connector_JST:JST_PH_B4B-PH-K_1x04_P2.00mm_Vertical" H 10250 1900 50  0001 C CNN
+F 1 "B4B-PH-K-S" H 10330 1801 50  0000 L CNN
+F 2 "Locator_Footprints:JST_PH_S4B-PH-SM4-TB_1x04-1MP_P2.00mm_Horizontal" H 10250 1900 50  0001 C CNN
 F 3 "~" H 10250 1900 50  0001 C CNN
 	1    10250 1900
 	1    0    0    -1
 $EndComp
-Text Label 9800 2100 0    50   ~ 0
-OUT2
-Text Label 9800 2000 0    50   ~ 0
-OUT4
+$Comp
+L power:GND #PWR0110
+U 1 1 5FE6563F
+P 4200 3000
+F 0 "#PWR0110" H 4200 2750 50  0001 C CNN
+F 1 "GND" H 4205 2827 50  0000 C CNN
+F 2 "" H 4200 3000 50  0001 C CNN
+F 3 "" H 4200 3000 50  0001 C CNN
+	1    4200 3000
+	1    0    0    -1
+$EndComp
+Text Notes 2100 3750 0    79   ~ 0
+5.5V Boost for logic and motor
 $EndSCHEMATC

Commit message: Added boost converter, continued layout
Parts:
- added C5, C8: 22uF, Capacitor_SMD:C_0805_2012Metric, symbol Device:C
- added C6: 1nF, Capacitor_SMD:C_0402_1005Metric, symbol Device:C
- added C7: 100nF, Capacitor_SMD:C_0402_1005Metric, symbol Device:C
- added JP1, JP2: VBB_Selection, Jumper:SolderJumper-3_P1.3mm_Bridged2Bar12_RoundedPad1.0x1.5mm, symbol Jumper:SolderJumper_3_Bridged12
- added L1: 4.7uH, Locator_Footprints:L_LQH44P, symbol Device:L
- added R5: 1.4M, Resistor_SMD:R_0603_1608Metric, symbol Device:R
- added R6: 412K, Resistor_SMD:R_0603_1608Metric, symbol Device:R
- C2: value 20uF -> 22uF
- C4, J1, J2, R1, R2: Assembly (none) -> DNP
- J3: value B4B-PH-K-S -> S4B-PH-SM4-TB; Link (none) -> https://www.digikey.de/product-detail/en/jst-sales-america-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; MPN (none) -> S4B-PH-SM4-TB(LF)(SN); Manufacturer (none) -> JST Sales America Inc.; Package (none) -> SMD; SPN (none) -> 455-1751-1-ND; description (none) -> Connector Header Surface Mount, Right Angle 4 position 0.07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
- U1: Link (none) -> https://eu.mouser.com/ProductDetail/NXP-Semiconductors/PCA9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; MPN (none) -> PCA9629APWJ; Manufacturer (none) -> NXP Semiconductors; Package (none) -> 16-TSSOP; SPN (none) -> 771-PCA9629APWJ; description (none) -> Bipolar, Unipolar Motor Driver CMOS I²C 16-TSSOP
- U2: Link (none) -> https://www.digikey.de/product-detail/en/allegro-microsyste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; MPN (none) -> A3909GLYTR-T; Manufacturer (none) -> Allegro MicroSystems; Package (none) -> 10-MSOP-EP; SPN (none) -> 620-1499-1-ND; description (none) -> Half Bridge (4) Driver DC Motors, General Purpose, Stepper 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
- U3: Link (none) -> https://www.mouser.de/ProductDetail/Maxim-Integrated/MAX172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; MPN (none) -> MAX17291ANT+; Manufacturer (none) -> Maxim Integrated; Package (none) -> TDFN; SPN (none) -> 700-MAX17291ANT+; description (none) -> Switching Voltage Regulators High-Voltage microPower Boost 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
Connections:
- net GND: now also U3.2 (AGND), U3.8 (GND), U3.9 (EP), C5.2, C6.2, C7.2, C8.2, R6.2
- net OUT1: now also J1.2 (Pin_2)
- net OUT2: now also J1.3 (Pin_3)
- net OUT3: now also J2.9 (Pin_9)
- net OUT4: now also J2.8 (Pin_8)
- net VBB: now also JP1.2 (C)
- net VDD: now also JP2.2 (C)
- net at U3.1 (LX): now also L1.2
- net VIN_BOOST: now reaches U3.3 (VIN)
- net VIN_BOOST: now also C5.1, C6.1, L1.1
- net EN: now reaches U3.4 (EN)
- net at U3.6 (FB): now also R5.2, R6.1
- net VOUT: now reaches U3.7 (VOUT)
- net VOUT: now also C7.1, C8.1, JP1.1 (A), JP2.1 (A), R5.1
- new net VIN_IC: JP2.3 (B)
- new net VIN_M: JP1.3 (B)
Other:
- note added: "Jumper Selection for use \nof internal or external power supply"
- moved on the sheet: U3

Commit message: Finished schematic and layout for now
Parts:
- JP2: value VBB_Selection -> VDD_Selection
- L1: footprint Locator_Footprints:L_LQH44P -> Inductor_SMD:L_1008_2520Metric; Link (none) -> https://www.digikey.de/product-detail/en/murata-electronics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; MPN (none) -> LQH2HPZ4R7MGRL; Manufacturer (none) -> Murata Electronics; Package (none) -> 1008 (2520 Metric); SPN (none) -> 490-15902-1-ND; description (none) -> 4.7µH Shielded Wirewound Inductor 1A 360mOhm Max 1008 (2520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
- R5, R6: footprint Resistor_SMD:R_0603_1608Metric -> Resistor_SMD:R_0402_1005Metric
Connections:
- net EN: now also J1.10 (Pin_10)
- net GND: now also J1.5 (Pin_5), J2.6 (Pin_6); no longer J1.10 (Pin_10)
- net INT: now also J2.5 (Pin_5)
- net OUT2: now also J2.9 (Pin_9); no longer J1.3 (Pin_3)
- net OUT3: now also J1.3 (Pin_3); no longer J2.9 (Pin_9)
- net P0: now also J1.8 (Pin_8)
- net P1: now also J1.7 (Pin_7)
- net P2: now also J1.6 (Pin_6)
- net RESET: now also J2.2 (Pin_2)
- net SCL: now also J2.4 (Pin_4)
- net SDA: now also J2.3 (Pin_3)
- net VIN_BOOST: now also J1.9 (Pin_9)
- net VIN_IC: now also J1.4 (Pin_4)
- net VIN_M: now also J2.7 (Pin_7)
Other:
- note added: "PCA9629A and motor are powered by the internal boost by \ndefault (5.5V). Cut and solder both jumpers to power the \ndriver (VIN_IC) and motor (VIN_M) through the external pin headers."
- moved on the sheet: JP1, JP2
Changed lines of the file:
@@
 Sheet 1 1
 Title "PCA9629A I²C Stepper Motor Controller Breakout Board"
-Date ""
+Date "2020-12-20"
 Rev "1"
 Comp "Igor Knippenberg"
@@
 	1    0    0    -1
 $EndComp
-Wire Wire Line
-	7800 2450 7350 2450
-$Comp
-L power:GND #PWR0109
-U 1 1 5FE45CE7
-P 7350 2450
-F 0 "#PWR0109" H 7350 2200 50  0001 C CNN
-F 1 "GND" H 7355 2277 50  0000 C CNN
-F 2 "" H 7350 2450 50  0001 C CNN
-F 3 "" H 7350 2450 50  0001 C CNN
-	1    7350 2450
-	1    0    0    -1
-$EndComp
 $Comp
 L Locator_Library:MAX17291 U3
@@
 F 0 "L1" V 2640 4150 50  0000 C CNN
 F 1 "4.7uH" V 2549 4150 50  0000 C CNN
-F 2 "Locator_Footprints:L_LQH44P" H 2450 4150 50  0001 C CNN
-F 3 "~" H 2450 4150 50  0001 C CNN
+F 2 "Inductor_SMD:L_1008_2520Metric" H 2450 4150 50  0001 C CNN
+F 3 "https://search.murata.co.jp/Ceramy/image/img/P02/JELF243A-9128.pdf" H 2450 4150 50  0001 C CNN
+F 4 "LQH2HPZ4R7MGRL" H 2450 4150 50  0001 C CNN "MPN"
+F 5 "Murata Electronics" H 2450 4150 50  0001 C CNN "Manufacturer"
+F 6 "490-15902-1-ND" H 2450 4150 50  0001 C CNN "SPN"
+F 7 "1008 (2520 Metric) " H 2450 4150 50  0001 C CNN "Package"
+F 8 "https://www.digikey.de/product-detail/en/murata-electronics/LQH2HPZ4R7MGRL/490-15902-1-ND/6800567" H 2450 4150 50  0001 C CNN "Link"
+F 9 " 4.7µH Shielded Wirewound Inductor 1A 360mOhm Max 1008 (2520 Metric) " H 2450 4150 50  0001 C CNN "description"
 	1    2450 4150
 	0    -1   -1   0
@@
 F 0 "R5" H 3570 4646 50  0000 L CNN
 F 1 "1.4M" H 3570 4555 50  0000 L CNN
-F 2 "Resistor_SMD:R_0603_1608Metric" V 3430 4600 50  0001 C CNN
+F 2 "Resistor_SMD:R_0402_1005Metric" V 3430 4600 50  0001 C CNN
 F 3 "https://www.koaspeer.com/pdfs/RK73H.pdf" H 3500 4600 50  0001 C CNN
 F 4 "https://www.mouser.de/ProductDetail/KOA-Speer/RK73H1JTTD1404F/?qs=%2Fha2pyFadujzle8xjALcvLDCByry4CFE4crEq4mQerqxX%252BnUx4sZzg%3D%3D" H 3500 4600 50  0001 C CNN "Link"
@@
 F 0 "R6" H 3570 4996 50  0000 L CNN
 F 1 "412K" H 3570 4905 50  0000 L CNN
-F 2 "Resistor_SMD:R_0603_1608Metric" V 3430 4950 50  0001 C CNN
+F 2 "Resistor_SMD:R_0402_1005Metric" V 3430 4950 50  0001 C CNN
 F 3 "https://eu.mouser.com/datasheet/2/219/RN73H-1843478.pdf" H 3500 4950 50  0001 C CNN
 F 4 "https://www.mouser.de/ProductDetail/KOA-Speer/RN73H1JTTD4123B25/?qs=%2Fha2pyFaduicUvIwceowioochi5c4TS6Cm3WX9AhKTnL0L4PmJpqqA%3D%3D" H 3500 4950 50  0001 C CNN "Link"
@@
 	1800 4450 2150 4450
 Wire Wire Line
-	6650 4200 6450 4200
+	5950 4250 5750 4250
 Wire Wire Line
 	7800 1650 7600 1650
@@
 OUT1
 Text Label 7600 1750 0    50   ~ 0
+OUT3
+Text Label 8800 1650 2    50   ~ 0
 OUT2
-Text Label 8800 1650 2    50   ~ 0
-OUT3
 Text Label 8800 1750 2    50   ~ 0
 OUT4
-Text Label 6450 4200 0    50   ~ 0
+Text Label 5750 4250 0    50   ~ 0
 VOUT
 Wire Wire Line
-	6850 4350 6850 4550
-Text Label 6850 4550 1    50   ~ 0
+	6150 4400 6150 4600
+Text Label 6150 4600 1    50   ~ 0
 VBB
 Wire Wire Line
-	7050 4200 7250 4200
-Text Label 7250 4200 2    50   ~ 0
+	6350 4250 6550 4250
+Text Label 6550 4250 2    50   ~ 0
 VIN_M
 Wire Notes Line
-	350  750  6800 750
+	600  600  7050 600
 Wire Wire Line
 	6350 2250 6600 2250
@@
 L Jumper:SolderJumper_3_Bridged12 JP1
 U 1 1 5FE7649B
-P 6850 4200
-F 0 "JP1" H 6850 4405 50  0000 C CNN
-F 1 "VBB_Selection" H 6850 4314 50  0000 C CNN
-F 2 "Jumper:SolderJumper-3_P1.3mm_Bridged2Bar12_RoundedPad1.0x1.5mm" H 6850 4200 50  0001 C CNN
-F 3 "~" H 6850 4200 50  0001 C CNN
-	1    6850 4200
-	1    0    0    -1
-$EndComp
-Wire Wire Line
-	6650 4950 6450 4950
-Text Label 6450 4950 0    50   ~ 0
+P 6150 4250
+F 0 "JP1" H 6150 4455 50  0000 C CNN
+F 1 "VBB_Selection" H 6150 4364 50  0000 C CNN
+F 2 "Jumper:SolderJumper-3_P1.3mm_Bridged2Bar12_RoundedPad1.0x1.5mm" H 6150 4250 50  0001 C CNN
+F 3 "~" H 6150 4250 50  0001 C CNN
+	1    6150 4250
+	1    0    0    -1
+$EndComp
+Wire Wire Line
+	7350 4250 7150 4250
+Text Label 7150 4250 0    50   ~ 0
 VOUT
 Wire Wire Line
-	6850 5100 6850 5300
-Text Label 6850 5300 1    50   ~ 0
+	7550 4400 7550 4600
+Text Label 7550 4600 1    50   ~ 0
 VDD
 Wire Wire Line
-	7050 4950 7250 4950
-Text Label 7250 4950 2    50   ~ 0
+	7750 4250 7950 4250
+Text Label 7950 4250 2    50   ~ 0
 VIN_IC
 $Comp
 L Jumper:SolderJumper_3_Bridged12 JP2
 U 1 1 5FE8918D
-P 6850 4950
-F 0 "JP2" H 6850 5155 50  0000 C CNN
-F 1 "VBB_Selection" H 6850 5064 50  0000 C CNN
-F 2 "Jumper:SolderJumper-3_P1.3mm_Bridged2Bar12_RoundedPad1.0x1.5mm" H 6850 4950 50  0001 C CNN
-F 3 "~" H 6850 4950 50  0001 C CNN
-	1    6850 4950
-	1    0    0    -1
-$EndComp
+P 7550 4250
+F 0 "JP2" H 7550 4455 50  0000 C CNN
+F 1 "VDD_Selection" H 7550 4364 50  0000 C CNN
+F 2 "Jumper:SolderJumper-3_P1.3mm_Bridged2Bar12_RoundedPad1.0x1.5mm" H 7550 4250 50  0001 C CNN
+F 3 "~" H 7550 4250 50  0001 C CNN
+	1    7550 4250
+	1    0    0    -1
+$EndComp
+Wire Wire Line
+	7800 2250 7600 2250
+Wire Wire Line
+	7800 2150 7600 2150
+Wire Wire Line
+	7800 2050 7600 2050
+Wire Wire Line
+	7800 1850 7600 1850
+Wire Wire Line
+	8600 1850 8800 1850
+Wire Wire Line
+	8600 2050 8800 2050
+Wire Wire Line
+	8600 2150 8800 2150
+Wire Wire Line
+	8600 2250 8800 2250
+Wire Wire Line
+	8600 2350 8800 2350
+Text Label 7400 2350 0    50   ~ 0
+VIN_BOOST
+Wire Wire Line
+	7400 2350 7800 2350
+Wire Wire Line
+	7800 2450 7600 2450
+Text Label 7600 2450 0    50   ~ 0
+EN
+Text Label 7600 2050 0    50   ~ 0
+P2
+Text Label 7600 2150 0    50   ~ 0
+P1
+Text Label 7600 2250 0    50   ~ 0
+P0
+Text Label 8800 1850 2    50   ~ 0
+VIN_M
+Text Label 7600 1850 0    50   ~ 0
+VIN_IC
+Wire Wire Line
+	7350 1950 7800 1950
+$Comp
+L power:GND #PWR0109
+U 1 1 5FE856A4
+P 7350 1950
+F 0 "#PWR0109" H 7350 1700 50  0001 C CNN
+F 1 "GND" H 7355 1777 50  0000 C CNN
+F 2 "" H 7350 1950 50  0001 C CNN
+F 3 "" H 7350 1950 50  0001 C CNN
+	1    7350 1950
+	1    0    0    -1
+$EndComp
+Text Label 8800 2050 2    50   ~ 0
+INT
+Text Label 8800 2150 2    50   ~ 0
+SCL
+Text Label 8800 2250 2    50   ~ 0
+SDA
+Text Label 8800 2350 2    50   ~ 0
+RESET
+Wire Wire Line
+	9050 1950 9050 2000
+Wire Wire Line
+	8600 1950 9050 1950
+$Comp
+L power:GND #PWR0116
+U 1 1 5FE93AD8
+P 9050 2000
+F 0 "#PWR0116" H 9050 1750 50  0001 C CNN
+F 1 "GND" H 9055 1827 50  0000 C CNN
+F 2 "" H 9050 2000 50  0001 C CNN
+F 3 "" H 9050 2000 50  0001 C CNN
+	1    9050 2000
+	1    0    0    -1
+$EndComp
+Text Notes 5600 5350 0    50   ~ 0
+PCA9629A and motor are powered by the internal boost by \ndefault (5.5V). Cut and solder both jumpers to power the \ndriver (VIN_IC) and motor (VIN_M) through the external pin headers.
 $EndSCHEMATC

Commit message: Bugfixes
Parts:
- C1: Link (none) -> https://www.digikey.com/product-detail/en/tdk-corporation/C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; MPN (none) -> C1005X5R1A475K050BC; Manufacturer (none) -> TDK Corporation; Package (none) -> 0402 (1005 Metric); SPN (none) -> 445-13820-1-ND; description (none) -> 4.7µF ±10% 10V Ceramic Capacitor X5R 0402 (1005 Metric)
- C2, C5, C8: Link (none) -> https://www.digikey.de/product-detail/en/samsung-electro-me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; MPN (none) -> CL21A226MAYNNNE; Manufacturer (none) -> Samsung Electro-Mechanics; Package (none) -> 0805 (2012 Metric); SPN (none) -> 1276-CL21A226MAYNNNECT-ND; description (none) -> 22µF ±20% 25V Ceramic Capacitor X5R 0805 (2012 Metric)
- C3, C7: Link (none) -> https://www.digikey.com/product-detail/en/murata-electronic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; MPN (none) -> GCM155R71C104JA55D; Manufacturer (none) -> Murata Electronics; Package (none) -> 0402 (1005 Metric); SPN (none) -> 490-16433-1-ND; description (none) -> 0.1µF ±5% 16V Ceramic Capacitor X7R 0402 (1005 Metric)
- C6: Link (none) -> https://www.digikey.de/product-detail/en/avx-corporation/04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; MPN (none) -> 0402YC102KAT2A; Manufacturer (none) -> AVX Corporation; Package (none) -> 0402 (1005 Metric); SPN (none) -> 478-6197-1-ND; description (none) -> 1000pF ±10% 16V Ceramic Capacitor X7R 0402 (1005 Metric)
- JP1, JP2: Assembly (none) -> DNP
- R3, R4: Link (none) -> https://www.digikey.com/product-detail/en/yageo/RC0402FR-07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; MPN (none) -> RC0402FR-0710KL; Manufacturer (none) -> Yageo; Package (none) -> 0402 (1005 Metric); SPN (none) -> 311-10.0KLRCT-ND; description (none) -> 10 kOhms ±1% 0.063W, 1/16W Chip Resistor 0402 (1005 Metric)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
- R5: footprint Resistor_SMD:R_0402_1005Metric -> Resistor_SMD:R_0603_1608Metric; Assembly DNP -> (none); Link https://www.mouser.de/ProductDetail/KOA-Speer/RK73H1JTTD140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 -> https://www.digikey.de/product-detail/en/koa-speer-electron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; Package 0603 -> 0603 (1608 Metric); SPN 660-RK73H1JTTD1404F -> 2019-RK73H1JTTD1404FCT-ND
- R6: footprint Resistor_SMD:R_0402_1005Metric -> Resistor_SMD:R_0603_1608Metric; Link https://www.mouser.de/ProductDetail/KOA-Speer/RN73H1JTTD412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 -> https://www.digikey.de/product-detail/en/koa-speer-electron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; Package 0603 -> 0603 (1608 Metric); SPN 660-RN73H1JTD4123B25 -> 2019-RN73H1JTTD4123B25CT-ND
- U1: Link https://eu.mouser.com/ProductDetail/NXP-Semiconductors/PCA9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 -> https://www.digikey.de/product-detail/en/nxp-usa-inc/PCA962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; SPN 771-PCA9629APWJ -> 568-11488-1-ND
Other:
- note added: "VIN: 1.8V - 5.5V"

Commit message: Layout modifications due to some bugs
h
Parts:
- removed JP2: VDD_Selection, Jumper:SolderJumper-3_P1.3mm_Bridged2Bar12_RoundedPad1.0x1.5mm, symbol Jumper:SolderJumper_3_Bridged12
- added D1, D2: LED, LED_SMD:LED_0603_1608Metric, symbol Device:LED
- added JP2, JP3: SolderJumper_2_Bridged, Jumper:SolderJumper-2_P1.3mm_Bridged2Bar_RoundedPad1.0x1.5mm, symbol Jumper:SolderJumper_2_Bridged
- added R7, R8: 10K, Resistor_SMD:R_0603_1608Metric, symbol Device:R
- R5: footprint Resistor_SMD:R_0603_1608Metric -> Resistor_SMD:R_0402_1005Metric; Link https://www.digikey.de/product-detail/en/koa-speer-electronics-inc/RK73H1JTTD1404F/2019-RK73H1JTTD1404FCT-ND/9847488 -> https://www.digikey.de/product-detail/en/koa-speer-electronics-inc/RK73H1ETTP1404F/2019-RK73H1ETTP1404FCT-ND/12367547; MPN RK73H1JTTD1404F -> RK73H1ETTP1404F; Package 0603 (1608 Metric) -> 0402 (1005 Metric); SPN 2019-RK73H1JTTD1404FCT-ND -> 2019-RK73H1ETTP1404FCT-ND; description 1.4 MOhms ±1% 0.1W, 1/10W Chip Resistor 0603 (1608 Metric) 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 -> 1.4 MOhms ±1% 0.1W, 1/10W Chip Resistor 0402 (1005 Metric) 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
- R6: footprint Resistor_SMD:R_0603_1608Metric -> Resistor_SMD:R_0402_1005Metric; Link https://www.digikey.de/product-detail/en/koa-speer-electron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 -> https://www.digikey.de/product-detail/de/panasonic-electron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; MPN RN73H1JTTD4123B25 -> ERJ-2RKF4123X; Manufacturer KOA Speer Electronics, Inc. -> Panasonic Electronic Components; Package 0603 (1608 Metric) -> 0402 (1005 Metric); SPN 2019-RN73H1JTTD4123B25CT-ND -> P412KLCT-ND; description 412 kOhms ±0.1% 0.1W, 1/10W Chip Resistor 0603 (1608 Metric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 -> 412 kOhms ±1% 0.1W, 1/10W Chip Resistor 0402 (1005 Metric) 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
- U3: footprint Locator_Footprints:MAX17291ATA+T -> Locator_Footprints:MAX17291ATA+; symbol Locator_Library:MAX17291 -> Locator_Library:MAX17291-WLP
Connections:
- net EN: now also J1.8 (Pin_8), U3.A3 (EN); no longer J1.10 (Pin_10), U3.4 (EN)
- net GND: now also J1.9 (Pin_9), J2.8 (Pin_8), U3.B1 (GND), D1.1 (K), D2.1 (K), JP2.1 (A), JP3.1 (A); no longer J1.1 (Pin_1), J1.5 (Pin_5), J2.10 (Pin_10), U1.5 (AD0), U1.6 (AD1), U3.2 (AGND), U3.8 (GND), U3.9 (EP)
- net OUT1: now also J1.1 (Pin_1); no longer J1.2 (Pin_2)
- net OUT2: now also J1.2 (Pin_2), J3.1 (Pin_1); no longer J2.9 (Pin_9), J3.4 (Pin_4)
- net OUT3: now also J2.10 (Pin_10), J3.4 (Pin_4); no longer J1.3 (Pin_3), J3.1 (Pin_1)
- net OUT4: now also J2.9 (Pin_9); no longer J2.8 (Pin_8)
- net P0: now also J1.7 (Pin_7); no longer J1.8 (Pin_8)
- net P1: now also J1.6 (Pin_6); no longer J1.7 (Pin_7)
- net P2: now also J1.5 (Pin_5); no longer J1.6 (Pin_6)
- net P3: now also R8.1
- net O1: now reaches U2.4 (IN3)
- net O1: now also U1.11 (OUT1); no longer U1.10 (OUT2)
- net O2: now reaches U2.2 (IN2)
- net O2: now also U1.10 (OUT2); no longer U1.11 (OUT1)
- net O0: now reaches U1.12 (OUT0), U2.1 (IN1)
- net O3: now reaches U1.9 (OUT3), U2.5 (IN4)
- net at L1.2: now also U3.A1 (LX); no longer U3.1 (LX)
- net at R5.2, R6.1: now also U3.B3 (FB); no longer U3.6 (FB)
- net VDD renamed VCC
- net VCC: now also C7.1, C8.1, JP1.1 (A), R5.1, U3.B2 (VOUT), R7.1
- net VIN_BOOST renamed VIN
- net VIN: now also J1.10 (Pin_10), U3.A2 (VIN); no longer J1.9 (Pin_9), U3.3 (VIN)
- net VIN_IC renamed AD0
- net AD0: now also U1.5 (AD0), JP3.2 (B)
- net VIN_M renamed VM
- removed net VOUT: C7.1, C8.1, JP1.1 (A), R5.1, U3.7 (VOUT)
- new net: D1.2 (A), R7.2
- new net: D2.2 (A), R8.2
- new net AD1: J1.3 (Pin_3), JP2.2 (B), U1.6 (AD1)
Other:
- note added: "4.5V - 5.5V"
- note added: "Black"
- note added: "Default I2C \naddress: 20h"
- note added: "For use with the "SM1507GB(100)" \nmini stepper motor"
- note added: "Internal/external motor \npower supply selection"
- note added: "LEDs"
- note added: "Orange"
- note added: "The motor is powered by the internal boost (5.5V). \nCut and solder the jumper to power the motor through \nthe external VM pin"
- note added: "White"
- note added: "Yellow"
- note removed: "I2C address: 40h"
- note removed: "Jumper Selection for use \nof internal or external power supply"
- note removed: "PCA9629A and motor are powered by the internal boost by \ndefault (5.5V). Cut and solder both jumpers to power the \ndriver (VIN_IC) and motor (VIN_M) through the external pin headers."
- note removed: "VDD: 4.5V - 5.5V"
- moved on the sheet: JP1
